Commit message: change damping value

File: unitree_description/a1_description/xacro/const.xacro (robot description, xacro)
@@ -29,5 +29,5 @@
     <xacro:property name="hip_offset" value="0.065"/>
     <!-- joint limits -->
-    <xacro:property name="damping" value="0"/>
+    <xacro:property name="damping" value="1.0"/>
     <xacro:property name="friction" value="0"/>
     <xacro:property name="hip_max" value="46"/>
