Commit message: add normal working version description file

File: unitree_description/a1_description/xacro/robot.xacro (robot description, xacro)
@@ -12,5 +12,5 @@
     <!-- <xacro:stairs stairs="15" xpos="0" ypos="0" zpos="0" /> -->
     <!-- Rollover Protection mode will add an additional stick on the top, use "true" or "false" to switch it. -->
-    <xacro:property name="rolloverProtection" value="false"/>
+    <xacro:property name="rolloverProtection" value="true"/>
     <!-- Debug mode will hung up the robot, use "true" or "false" to switch it. -->
     <xacro:if value="$(arg DEBUG)">
@@ -124,5 +124,5 @@
         <origin rpy="0 0 0" xyz="${-leg_offset_x} ${leg_offset_y} 0"/>
     </xacro:leg>
-    <!-- <xacro:unless value="$(arg use_gazebo)">
+    <xacro:unless value="$(arg use_gazebo)">
         <ros2_control name="a1_ros2_control_settings" type="system">
             <hardware>
@@ -162,10 +162,10 @@
             </sensor>
         </ros2_control>
-    </xacro:unless> -->
+    </xacro:unless>
     <xacro:if value="$(arg use_gazebo)">
         <ros2_control name="a1_ros2_control_settings" type="system">
             <hardware>
                 <plugin>unitree_gazebo/UnitreeGazeboSystem</plugin>
-                <!-- <plugin>gazebo_ros2_control/GazeboSystem</plugin> -->
+                <!-- <plugin>gazebo_ros2_control/GazeboSystem</plugin> since we have modified version in unitree_gazebo-->
             </hardware>
             <xacro:leg_ros2_control leg_name="FL"/>
@@ -204,5 +204,4 @@
         <gazebo>
             <plugin filename="libgazebo_ros2_control.so" name="gazebo_ros2_control">
-            <!-- <plugin name="gazebo_ros2_control" filename="libgazebo_ros2_control.so"> -->
                 <robot_sim_type>    </robot_sim_type>
                 <parameters>$(find unitree_controller)/config/a1_gazebo_controllers.yaml</parameters>
