Commit message: add python code, TODO: check trunk position in moving_body and visualization

File: skiing_test/oop_skiing/a1.urdf (robot description, URDF)
Before this commit: robot a1_description, 23 links, 22 joints
Joints:
- joint FL_hip_fixed: origin xyz=0 0.081 0 rpy=0 0 0 -> xyz=0 0.0838 0 rpy=0 0 0
- joint FR_calf_joint: origin xyz=0 0 -0.2 rpy=0 0 0 -> xyz=0 0 -0.22 rpy=0 0 0
- joint FR_foot_fixed: origin xyz=0 0 -0.2 rpy=0 0 0 -> xyz=0 0 -0.22 rpy=0 0 0
- joint FR_hip_fixed: origin xyz=0 -0.081 0 rpy=0 0 0 -> xyz=0 -0.0838 0 rpy=0 0 0
- joint RL_hip_fixed: origin xyz=0 0.081 0 rpy=0 0 0 -> xyz=0 0.0838 0 rpy=0 0 0
- joint RR_hip_fixed: origin xyz=0 -0.081 0 rpy=0 0 0 -> xyz=0 -0.0838 0 rpy=0 0 0
